File: Hardware/KiCad/ioBoard.kicad_pcb (KiCad board)
At the start: 4 copper layers, 70 x 143 mm, 199 parts, among them J10 Micro_SD_Card, J11 8P8C_LED_Shielded, J12 MPT 0.5/3-2.54, J13 MPT 0.5/3-2.54, J14 MPT 0.5/3-2.54, J15 MPT 0.5/3-2.54, J16 MPT 0.5/3-2.54, J17 MPT 0.5/3-2.54, J18 MPT 0.5/3-2.54, J19 MPT 0.5/3-2.54, J20 MPT 0.5/2-2.54, J21 MPT 0.5/3-2.54, J22 MPT 0.5/3-2.54, J23 MPT 0.5/3-2.54, J24 MPT 0.5/3-2.54, J25 MPT 0.5/3-2.54, J26 MPT 0.5/3-2.54, J27 MPT 0.5/3-2.54, J28 MPT 0.5/3-2.54, J29 MPT 0.5/3-2.54, J30 MPT 0.5/3-2.54, J31 MPT 0.5/3-2.54, J32 MPT 0.5/3-2.54, J33 USB_B_Micro, J34 MPT 0.5/3-2.54, J9 ICSP, K1 G5Q-1EU, K2 G5Q-1EU, K3 G5Q-1EU, K4 G5Q-1EU, K5 G5Q-1EU, K6 G5Q-1EU, K7 G5Q-1EU, K8 G5Q-1EU, Q1 RU1C001UNTCL, Q2 RU1C001UNTCL, Q3 RU1C001UNTCL, Q4 RU1C001UNTCL, Q5 RU1C001UNTCL, Q6 RU1C001UNTCL, Q7 RU1C001UNTCL, Q8 RU1C001UNTCL, Q9 RU1C001UNTCL, SW1 SW_DPST, U1 ATmega2560, U10 SFH617A-1, U11 SFH617A-1, U12 SFH617A-1, U13 SFH617A-1, U14 SFH617A-1, U15 LM2904, U16 SFH617A-1, U17 SFH617A-1, U18 SFH617A-1, U19 DS1307+, U2 74AHC1G125, U20 MIC5504-3.3YM5, U21 AP1509, U22 FT232RL, U3 74AHC1G125, U4 74AHC1G125, U5 74AHC1G125, U6 W5100, U7 SFH617A-1, U8 SFH617A-1, U9 SFH617A-1, Y1 16MHz, Y2 25MHz, Y3 32.768KHz

Commit message: V1.2
Parts:
- added C36: 100nF, Capacitor_SMD:C_0603_1608Metric, F.Cu at (130.1, 100.5)
- added R62: 10K, Resistor_SMD:R_0603_1608Metric, F.Cu at (93.4, 176.7)
- added R63: 10K, Resistor_SMD:R_0603_1608Metric, F.Cu at (93.4, 190.6)
- added R64: 10K, Resistor_SMD:R_0603_1608Metric, F.Cu at (110.9, 155.7)
- added R65: 10K, Resistor_SMD:R_0603_1608Metric, F.Cu at (110.9, 169.5)
- added R66: 10K, Resistor_SMD:R_0603_1608Metric, F.Cu at (110.9, 183.2)
- added R67: 10K, Resistor_SMD:R_0603_1608Metric, F.Cu at (110.9, 197.2)
- BT1: footprint my_footprint:BatteryHolder_Keystone_103_1x20mm -> pbo_footprint:BatteryHolder_Keystone_103_1x20mm
- D1: footprint my_footprint:D_Sub_SMA -> pbo_footprint:D_Sub_SMA
- J11: footprint my_footprint:RJ45_Stewart_SS_74301_001 -> pbo_footprint:RJ45_Stewart_SS_74301_001
- J12, J13, J14, J15, J16, J17, J18, J19: footprint TerminalBlock_Phoenix:TerminalBlock_Phoenix_MPT-0,5-3-2.54_1x03_P2.54mm_Horizontal -> pbo_footprint:TerminalBlock_Phoenix_MPT-0,5-3-2.54_1x03_P2.54mm_Horizontal
- J20, J21, J22, J23, J24, J25, J26, J27, J28, J29, J30, J31, J32, J34: footprint my_footprint:TerminalBlock_Phoenix_MPT-0,5-2-2.54_1x02_P2.54mm_Horizontal -> pbo_footprint:TerminalBlock_Phoenix_MPT-0,5-2-2.54_1x02_P2.54mm_Horizontal
- J33: footprint Connector_USB:USB_Micro-B_Amphenol_10103594-0001LF_Horizontal -> pbo_footprint:USB_Micro-B_Amphenol_110118192-0001LF_Horizontal
- J9: footprint my_footprint:2178710-6_Micro-MaTch_TE_CONNECTIVITY -> Connector_PinHeader_2.54mm:PinHeader_2x03_P2.54mm_Vertical
- K1, K2, K3, K4, K5, K6, K7, K8: footprint my_footprint:Relay_SPDT_Omron-G5Q-1 -> pbo_footprint:Relay_SPDT_Omron-G5Q-1
- L1: footprint my_footprint:L_Bourns-SRU8043 -> pbo_footprint:L_Bourns-SRU8043
- R14: value 100 -> 10K
- R57: value 1K -> 10K
- R58: value 3K -> 10K
- R61: value 10K -> 1K5
- SW1: footprint Button_Switch_SMD:SW_SPST_B3S-1000 -> pbo_footprint:SW_SPST_B3S-1000
- U16: value SFH617A-1 -> SFH620A
- Y1: footprint Crystal:Crystal_SMD_3225-4Pin_3.2x2.5mm -> pbo_footprint:Crystal_SMD_2520-4Pin_2.5x2.0mm
- Y2: footprint Crystal:Crystal_SMD_3225-4Pin_3.2x2.5mm -> Crystal:Crystal_SMD_2016-4Pin_2.0x1.6mm
- Y3: footprint Crystal:Crystal_SMD_3225-4Pin_3.2x2.5mm -> Crystal:Crystal_SMD_3215-2Pin_3.2x1.5mm
- moved R58 31.0 mm to (93.4, 162.7), turned to 180 degrees
- moved R57 24.6 mm to (93.4, 148.7), turned to 180 degrees
- moved J9 2.28 mm to (107.4, 121.3), turned to 270 degrees
- moved C26 1.25 mm to (90.2, 137.1), turned to 270 degrees
- moved C25 1.24 mm to (90.2, 144.7), turned to 270 degrees
- moved Y2 0.40 mm to (128.2, 82.9)
- moved J33 0.29 mm to (136.6, 84.7)
- moved Y3 0.10 mm to (133.5, 131.2), turned to 45 degrees
Connections:
- J9 pad 1: /MISO -> /ICSP_MISO
- J9 pad 3: /SCK -> /ICSP_SCK
- J9 pad 4: /MOSI -> /ICSP_MOSI
- J9 pad 6: Net-(J9-Pad6) -> Earth
- R4 pad 1: Net-(R4-Pad1) -> /ICSP_MISO
- R5 pad 1: Net-(R5-Pad1) -> /ICSP_SCK
- R57 pad 1: Earth -> /STOR_3
- R57 pad 2: Net-(R57-Pad2) -> Earth
- R58 pad 1: Net-(R57-Pad2) -> /STOR_6
- R58 pad 2: Net-(D29-Pad1) -> Earth
- R6 pad 1: Net-(R6-Pad1) -> /ICSP_MOSI
- U1 pad 20: Net-(R5-Pad1) -> /ICSP_SCK
- U1 pad 21: Net-(R6-Pad1) -> /ICSP_MOSI
- U1 pad 22: Net-(R4-Pad1) -> /ICSP_MISO
- U2 pad 1: Net-(U2-Pad1) -> Earth
- U21 pad 3: Net-(R57-Pad2) -> +5V
- U3 pad 1: Net-(U3-Pad1) -> Earth
- Y2 pad 2: Net-(C24-Pad2) -> Net-(Y2-Pad2)
- Y2 pad 3: (no net) -> Net-(C24-Pad2)
Routing:
- net /MOSI: track 74.1 -> 18.9 mm
- net /SCK: track 71.2 -> 16.3 mm
- net /ICSP_MOSI: track 0.00 -> 54.0 mm, vias 0 -> 1
- net /ICSP_SCK: track 0.00 -> 52.9 mm, vias 0 -> 1
- net /ICSP_MISO: track 0.00 -> 45.9 mm, vias 0 -> 1
- net /MISO: track 77.2 -> 32.7 mm
- net Earth: track 112.7 -> 103.7 mm, vias 110 -> 107
- net +5V: track 51.3 -> 58.0 mm, vias 23 -> 24
- net +12V: track 78.3 -> 83.8 mm
- net Net-(U19-Pad1): track 8.52 -> 3.19 mm
- net Net-(R4-Pad1): track 4.98 -> 0.00 mm
- net Net-(R57-Pad2): track 4.65 -> 0.00 mm
- net Net-(R5-Pad1): track 3.88 -> 0.00 mm
- net Net-(R6-Pad1): track 3.88 -> 0.00 mm
- net Net-(C24-Pad2): track 4.64 -> 7.27 mm
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Other:
- board text added: "+"
- board text added: "-"
- board text added: "Design by P. Boissard for Crozitech"
